File: iso-usb2pwrd.kicad_pcb (KiCad board)
At the start: 2 copper layers, 35 x 18 mm, 32 parts, among them J1 USB_C_Receptacle_USB2.0_14P, J2 USB_C_Receptacle_USB2.0_14P, U1 ADuM3165, U2 R05C1TF05S, U3 TPS25820, Y1 24Mhz

Commit message: add board rev
Parts:
- D1, D2: value D_TVS_Dual_AAC -> ESD752
Other:
- board text added: "R1.0.0"
Changed lines of the file:
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@@
 			)
 		)
-		(property "MPN" ""
+		(property "MPN" "GCM155R71H104KE02D"
 			(at 0 0 -90)
 			(unlocked yes)
@@
 			)
 		)
-		(property "MPN" ""
+		(property "MPN" "GCM155R71H104KE02D"
 			(at 0 0 -90)
 			(unlocked yes)
@@
 			)
 		)
-		(property "MPN" ""
+		(property "MPN" "RC0402FR-075K1L"
 			(at 0 0 0)
 			(unlocked yes)
@@
 			)
 		)
-		(property "MPN" ""
+		(property "MPN" "GCM155R71H104KE02D"
 			(at 0 0 -90)
 			(unlocked yes)
@@
 			)
 		)
-		(property "MPN" ""
+		(property "MPN" "RC0402FR-07100KL"
 			(at 0 0 -90)
 			(unlocked yes)
@@
 			)
 		)
-		(property "MPN" ""
+		(property "MPN" "RC0402FR-075K1L"
 			(at 0 0 -90)
 			(unlocked yes)
@@
 			)
 		)
-		(property "Value" "D_TVS_Dual_AAC"
+		(property "Value" "ESD752"
 			(at -0.05 2.05 180)
 			(layer "F.Fab")
@@
 			)
 		)
-		(property "MPN" ""
+		(property "MPN" "ESD752DCKR"
 			(at 0 0 180)
 			(unlocked yes)
@@
 			)
 		)
-		(property "MPN" ""
+		(property "MPN" "0402N150J250CT"
 			(at 0 0 180)
 			(unlocked yes)
@@
 			)
 		)
-		(property "MPN" ""
+		(property "MPN" "GCM155R71H104KE02D"
 			(at 0 0 -90)
 			(unlocked yes)
@@
 			)
 		)
-		(property "MPN" ""
+		(property "MPN" "GCM155R71H104KE02D"
 			(at 0 0 -90)
 			(unlocked yes)
@@
 			)
 		)
-		(property "Value" "D_TVS_Dual_AAC"
+		(property "Value" "ESD752"
 			(at -0.05 2.05 0)
 			(layer "F.Fab")
@@
 			)
 		)
-		(property "MPN" ""
+		(property "MPN" "ESD752DCKR"
 			(at 0 0 0)
 			(unlocked yes)
@@
 			)
 		)
-		(property "MPN" ""
+		(property "MPN" "RC0402FR-075K1L"
 			(at 0 0 -90)
 			(unlocked yes)
@@
 			)
 		)
-		(property "MPN" ""
+		(property "MPN" "0402N150J250CT"
 			(at 0 0 -90)
 			(unlocked yes)
@@
 			)
 		)
-		(property "MPN" ""
+		(property "MPN" "RC0402FR-075K1L"
 			(at 0 0 -90)
 			(unlocked yes)
@@
 			)
 		)
-		(property "MPN" ""
+		(property "MPN" "RC0402FR-075K1L"
 			(at 0 0 180)
 			(unlocked yes)
@@
 			)
 		)
-		(property "MPN" ""
+		(property "MPN" "GCM155R71H104KE02D"
 			(at 0 0 -90)
 			(unlocked yes)
@@
 		)
 	)
+	(gr_text "R1.0.0"
+		(at 101.67 69.355 90)
+		(layer "B.SilkS")
+		(effects
+			(font
+				(size 1.3 1.3)
+				(thickness 0.2)
+			)
+			(justify top mirror)
+		)
+	)
