File: iso-usb2pwrd.kicad_sch (KiCad schematic)
At the start: 32 parts, among them J1 USB_C_Receptacle_USB2.0_14P, J2 USB_C_Receptacle_USB2.0_14P, U1 ADuM3165, U2 R05C1TF05S, U3 TPS25820, Y1 24Mhz

Commit message: add board rev
Parts:
- C10, C2, C4, C7, C8, C9: MPN (none) -> GCM155R71H104KE02D
- C5, C6: MPN (none) -> 0402N150J250CT
- D1, D2: value D_TVS_Dual_AAC -> ESD752; MPN (none) -> ESD752DCKR
- R1, R2, R4, R5, R6: MPN (none) -> RC0402FR-075K1L
- R3: MPN (none) -> RC0402FR-07100KL
Other:
- moved on the sheet: D1
